File: PCB Files/square Rev1.brd (EAGLE design)
At the start: 47 x 30.5 mm, 42 parts, among them U1 LM1117MP-5.0, Y1 16MHz

Commit message: some pcb adjustments
Routing:
- net N$3: track 17.3 -> 18.2 mm
- net 5V_PROTECTED: track 52.6 -> 53.4 mm
Changed lines of the file:
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@@
 <grid distance="50" unitdist="mil" unit="mil" style="lines" multiple="1" display="no" altdistance="5" altunitdist="mil" altunit="mil"/>
 <layers>
-<layer number="1" name="Top" color="4" fill="1" visible="no" active="yes"/>
+<layer number="1" name="Top" color="4" fill="1" visible="yes" active="yes"/>
 <layer number="2" name="Route2" color="1" fill="3" visible="no" active="no"/>
 <layer number="3" name="Route3" color="4" fill="3" visible="no" active="no"/>
@@
 <layer number="19" name="Unrouted" color="6" fill="1" visible="yes" active="yes"/>
 <layer number="20" name="Dimension" color="24" fill="1" visible="yes" active="yes"/>
-<layer number="21" name="tPlace" color="7" fill="1" visible="no" active="yes"/>
+<layer number="21" name="tPlace" color="7" fill="1" visible="yes" active="yes"/>
 <layer number="22" name="bPlace" color="7" fill="1" visible="yes" active="yes"/>
-<layer number="23" name="tOrigins" color="15" fill="1" visible="no" active="yes"/>
+<layer number="23" name="tOrigins" color="15" fill="1" visible="yes" active="yes"/>
 <layer number="24" name="bOrigins" color="15" fill="1" visible="yes" active="yes"/>
-<layer number="25" name="tNames" color="7" fill="1" visible="no" active="yes"/>
+<layer number="25" name="tNames" color="7" fill="1" visible="yes" active="yes"/>
 <layer number="26" name="bNames" color="7" fill="1" visible="yes" active="yes"/>
 <layer number="27" name="tValues" color="7" fill="1" visible="no" active="yes"/>
@@
 <layer number="37" name="tTest" color="7" fill="1" visible="no" active="yes"/>
 <layer number="38" name="bTest" color="7" fill="1" visible="no" active="yes"/>
-<layer number="39" name="tKeepout" color="4" fill="11" visible="no" active="yes"/>
+<layer number="39" name="tKeepout" color="4" fill="11" visible="yes" active="yes"/>
 <layer number="40" name="bKeepout" color="1" fill="11" visible="yes" active="yes"/>
-<layer number="41" name="tRestrict" color="4" fill="10" visible="no" active="yes"/>
+<layer number="41" name="tRestrict" color="4" fill="10" visible="yes" active="yes"/>
 <layer number="42" name="bRestrict" color="1" fill="10" visible="yes" active="yes"/>
 <layer number="43" name="vRestrict" color="2" fill="10" visible="no" active="yes"/>
@@
 <layer number="49" name="Reference" color="7" fill="1" visible="no" active="yes"/>
 <layer number="50" name="dxf" color="7" fill="1" visible="no" active="no"/>
-<layer number="51" name="tDocu" color="7" fill="1" visible="no" active="yes"/>
+<layer number="51" name="tDocu" color="7" fill="1" visible="yes" active="yes"/>
 <layer number="52" name="bDocu" color="7" fill="1" visible="yes" active="yes"/>
 <layer number="53" name="tGND_GNDA" color="7" fill="9" visible="no" active="no"/>
@@
 </element>
 <element name="RAW" library="testpad" library_urn="urn:adsk.eagle:library:385" package="B2,54" package3d_urn="urn:adsk.eagle:package:27948/1" value="TPB2,54" x="1.778" y="19.05" smashed="yes" rot="MR180">
-<attribute name="NAME" x="0.381" y="22.86" size="0.762" layer="26" font="vector" ratio="10" rot="MR270"/>
+<attribute name="NAME" x="0.381" y="20.32" size="0.762" layer="26" font="vector" ratio="10" rot="MR270"/>
 <attribute name="TP_SIGNAL_NAME" value="" x="0.508" y="22.225" size="1" layer="38" rot="MR180"/>
 <attribute name="VALUE" x="0.508" y="20.447" size="0.0254" layer="28" rot="MR180"/>
 </element>
 <element name="GND" library="testpad" library_urn="urn:adsk.eagle:library:385" package="B2,54" package3d_urn="urn:adsk.eagle:package:27948/1" value="TPB2,54" x="-3.048" y="19.05" smashed="yes" rot="MR0">
-<attribute name="NAME" x="-2.159" y="22.86" size="0.762" layer="26" font="vector" ratio="10" rot="MR270"/>
+<attribute name="NAME" x="-4.699" y="20.32" size="0.762" layer="26" font="vector" ratio="10" rot="MR270"/>
 <attribute name="TP_SIGNAL_NAME" value="" x="-1.778" y="15.875" size="1" layer="38" rot="MR0"/>
 <attribute name="VALUE" x="-1.778" y="17.653" size="0.0254" layer="28" rot="MR0"/>
@@
 <wire x1="14.4" y1="15.21" x2="14.3232" y2="15.16614375" width="0.2" layer="1"/>
 <wire x1="20.88" y1="20.61" x2="20.9595375" y2="20.6711125" width="0.2" layer="1"/>
-<wire x1="30.96" y1="12.06" x2="30.96" y2="11.43" width="0.2" layer="16"/>
-<wire x1="23.85" y1="19.17" x2="30.96" y2="12.06" width="0.2" layer="16"/>
-<wire x1="22.59" y1="19.17" x2="23.85" y2="19.17" width="0.2" layer="16"/>
+<wire x1="25.12" y1="19.17" x2="22.59" y2="19.17" width="0.2" layer="16"/>
 <wire x1="17.73" y1="24.03" x2="20.925" y2="20.835" width="0.2" layer="16"/>
 <wire x1="20.925" y1="20.835" x2="22.59" y2="19.17" width="0.2" layer="16"/>
@@
 <wire x1="21.78" y1="21.6" x2="21.87" y2="21.6" width="0.2" layer="1"/>
 <via x="21.78" y="21.6" extent="1-16" drill="0.35"/>
+<wire x1="31.02" y1="11.43" x2="31.02" y2="13.43" width="0.2032" layer="16"/>
+<wire x1="25.28" y1="19.17" x2="25.12" y2="19.17" width="0.2032" layer="16"/>
+<wire x1="31.02" y1="13.43" x2="25.4" y2="19.05" width="0.2032" layer="16"/>
+<wire x1="25.4" y1="19.05" x2="25.28" y2="19.17" width="0.1524" layer="16"/>
 </signal>
 <signal name="TXD">
@@
 <wire x1="12.121571875" y1="20.61" x2="12.15" y2="20.61" width="0.1524" layer="1"/>
 <contactref element="1K1" pad="2"/>
-<wire x1="15.66" y1="19.05" x2="15.36" y2="19.35" width="0.1524" layer="16"/>
-<wire x1="15.36" y1="19.35" x2="13.86" y2="19.35" width="0.1524" layer="16"/>
+<wire x1="15.66" y1="19.05" x2="15.36" y2="19.35" width="0.2032" layer="16"/>
+<wire x1="15.36" y1="19.35" x2="13.86" y2="19.35" width="0.2032" layer="16"/>
 </signal>
 <signal name="RXD">
@@
 <wire x1="12.69" y1="21.172940625" x2="12.69" y2="21.15" width="0.1524" layer="1"/>
 <contactref element="1K" pad="2"/>
-<wire x1="13.5" y1="20.34" x2="14.75" y2="21.59" width="0.1524" layer="16"/>
-<wire x1="14.75" y1="21.59" x2="15.66" y2="21.59" width="0.1524" layer="16"/>
+<wire x1="13.5" y1="20.34" x2="14.75" y2="21.59" width="0.2032" layer="16"/>
+<wire x1="14.75" y1="21.59" x2="15.66" y2="21.59" width="0.2032" layer="16"/>
 </signal>
 <signal name="SCL">
@@
 <contactref element="1K1" pad="1"/>
 <wire x1="29.02" y1="11.43" x2="29.21" y2="11.62" width="0.1524" layer="16"/>
-<wire x1="29.21" y1="11.62" x2="29.21" y2="12.7" width="0.1524" layer="16"/>
-<wire x1="29.21" y1="12.7" x2="27.94" y2="13.97" width="0.1524" layer="16"/>
-<wire x1="27.94" y1="13.97" x2="24.13" y2="13.97" width="0.1524" layer="16"/>
-<wire x1="24.13" y1="13.97" x2="19.05" y2="19.05" width="0.1524" layer="16"/>
-<wire x1="19.05" y1="19.05" x2="17.36" y2="19.05" width="0.1524" layer="16"/>
+<wire x1="29.21" y1="11.62" x2="29.21" y2="12.7" width="0.2032" layer="16"/>
+<wire x1="29.21" y1="12.7" x2="27.94" y2="13.97" width="0.2032" layer="16"/>
+<wire x1="27.94" y1="13.97" x2="24.13" y2="13.97" width="0.2032" layer="16"/>
+<wire x1="24.13" y1="13.97" x2="19.05" y2="19.05" width="0.2032" layer="16"/>
+<wire x1="19.05" y1="19.05" x2="17.36" y2="19.05" width="0.2032" layer="16"/>
 </signal>
 <signal name="N$3">
@@
 <contactref element="1K" pad="1"/>
 <wire x1="30.02" y1="11.43" x2="30.0162" y2="11.7762" width="0.1524" layer="16"/>
-<wire x1="30.0162" y1="11.7762" x2="29.5562" y2="12.79560625" width="0.1524" layer="16"/>
-<wire x1="29.5562" y1="12.79560625" x2="27.11180625" y2="15.24" width="0.1524" layer="16"/>
-<wire x1="27.11180625" y1="15.24" x2="24.13" y2="15.24" width="0.1524" layer="16"/>
-<wire x1="24.13" y1="15.24" x2="17.78" y2="21.59" width="0.1524" layer="16"/>
-<wire x1="17.78" y1="21.59" x2="17.36" y2="21.59" width="0.1524" layer="16"/>
+<wire x1="27.94" y1="15.24" x2="24.13" y2="15.24" width="0.2032" layer="16"/>
+<wire x1="24.13" y1="15.24" x2="17.78" y2="21.59" width="0.2032" layer="16"/>
+<wire x1="17.78" y1="21.59" x2="17.36" y2="21.59" width="0.2032" layer="16"/>
+<wire x1="30.02" y1="11.43" x2="30.02" y2="13.16" width="0.2032" layer="16"/>
+<wire x1="30.02" y1="13.16" x2="27.94" y2="15.24" width="0.2032" layer="16"/>
 </signal>
 </signals>
