File: PCB Files/square Rev2.brd (EAGLE design)
At the start: 47 x 30.5 mm, 36 parts, among them Y1 16MHz

Commit message: Minor PCB update
Parts:
- added 5V, G: TPB1,27, testpad:B1,27
Connections:
- net 5V_PROTECTED: now also 5V.TP
- net GND: now also G.TP
Routing:
- net 5V_PROTECTED: track 49.6 -> 53.8 mm, vias 1 -> 2
Changed lines of the file:
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@@
 <grid distance="50" unitdist="mil" unit="mil" style="lines" multiple="1" display="no" altdistance="5" altunitdist="mil" altunit="mil"/>
 <layers>
-<layer number="1" name="Top" color="4" fill="1" visible="yes" active="yes"/>
+<layer number="1" name="Top" color="4" fill="1" visible="no" active="yes"/>
 <layer number="2" name="Route2" color="1" fill="3" visible="no" active="no"/>
 <layer number="3" name="Route3" color="4" fill="3" visible="no" active="no"/>
@@
 <layer number="14" name="Route14" color="1" fill="6" visible="no" active="no"/>
 <layer number="15" name="Route15" color="4" fill="6" visible="no" active="no"/>
-<layer number="16" name="Bottom" color="1" fill="1" visible="no" active="yes"/>
+<layer number="16" name="Bottom" color="1" fill="1" visible="yes" active="yes"/>
 <layer number="17" name="Pads" color="2" fill="1" visible="yes" active="yes"/>
 <layer number="18" name="Vias" color="2" fill="1" visible="yes" active="yes"/>
 <layer number="19" name="Unrouted" color="6" fill="1" visible="yes" active="yes"/>
 <layer number="20" name="Dimension" color="24" fill="1" visible="yes" active="yes"/>
-<layer number="21" name="tPlace" color="7" fill="1" visible="yes" active="yes"/>
-<layer number="22" name="bPlace" color="7" fill="1" visible="no" active="yes"/>
-<layer number="23" name="tOrigins" color="15" fill="1" visible="yes" active="yes"/>
-<layer number="24" name="bOrigins" color="15" fill="1" visible="no" active="yes"/>
-<layer number="25" name="tNames" color="7" fill="1" visible="yes" active="yes"/>
-<layer number="26" name="bNames" color="7" fill="1" visible="no" active="yes"/>
+<layer number="21" name="tPlace" color="7" fill="1" visible="no" active="yes"/>
+<layer number="22" name="bPlace" color="7" fill="1" visible="yes" active="yes"/>
+<layer number="23" name="tOrigins" color="15" fill="1" visible="no" active="yes"/>
+<layer number="24" name="bOrigins" color="15" fill="1" visible="yes" active="yes"/>
+<layer number="25" name="tNames" color="7" fill="1" visible="no" active="yes"/>
+<layer number="26" name="bNames" color="7" fill="1" visible="yes" active="yes"/>
 <layer number="27" name="tValues" color="7" fill="1" visible="no" active="yes"/>
 <layer number="28" name="bValues" color="7" fill="1" visible="no" active="yes"/>
@@
 <layer number="37" name="tTest" color="7" fill="1" visible="no" active="yes"/>
 <layer number="38" name="bTest" color="7" fill="1" visible="no" active="yes"/>
-<layer number="39" name="tKeepout" color="4" fill="11" visible="yes" active="yes"/>
-<layer number="40" name="bKeepout" color="1" fill="11" visible="no" active="yes"/>
-<layer number="41" name="tRestrict" color="4" fill="10" visible="yes" active="yes"/>
-<layer number="42" name="bRestrict" color="1" fill="10" visible="no" active="yes"/>
+<layer number="39" name="tKeepout" color="4" fill="11" visible="no" active="yes"/>
+<layer number="40" name="bKeepout" color="1" fill="11" visible="yes" active="yes"/>
+<layer number="41" name="tRestrict" color="4" fill="10" visible="no" active="yes"/>
+<layer number="42" name="bRestrict" color="1" fill="10" visible="yes" active="yes"/>
 <layer number="43" name="vRestrict" color="2" fill="10" visible="no" active="yes"/>
 <layer number="44" name="Drills" color="7" fill="1" visible="no" active="yes"/>
@@
 <layer number="49" name="Reference" color="7" fill="1" visible="no" active="yes"/>
 <layer number="50" name="dxf" color="7" fill="1" visible="no" active="no"/>
-<layer number="51" name="tDocu" color="7" fill="1" visible="yes" active="yes"/>
-<layer number="52" name="bDocu" color="7" fill="1" visible="no" active="yes"/>
+<layer number="51" name="tDocu" color="7" fill="1" visible="no" active="yes"/>
+<layer number="52" name="bDocu" color="7" fill="1" visible="yes" active="yes"/>
 <layer number="53" name="tGND_GNDA" color="7" fill="9" visible="no" active="no"/>
 <layer number="54" name="bGND_GNDA" color="1" fill="9" visible="no" active="no"/>
@@
 <wire x1="3.81" y1="6.35" x2="3.81" y2="16.51" width="0.1524" layer="20"/>
 <wire x1="3.81" y1="16.51" x2="-6.35" y2="16.51" width="0.1524" layer="20"/>
-<text x="21.59" y="31.75" size="0.762" layer="22" font="vector" ratio="10" rot="MR180">ISCP: GND-SCK-5V-MO-MI-RES</text>
+<text x="20.32" y="31.75" size="0.762" layer="22" font="vector" ratio="10" rot="MR180">ISCP: GND-SCK-5V-MO-MI-RES</text>
 </plain>
 <attributes>
@@
 <elements>
 <element name="ATMEGA" library="SparkFun-IC-Microcontroller" library_urn="urn:adsk.eagle:library:525" package="TQFP32-08" package3d_urn="urn:adsk.eagle:package:38945/1" value="ATMEGA328P_TQFP" x="16.51" y="19.05" smashed="yes" rot="R45">
-<attribute name="NAME" x="16.959015625" y="18.600984375" size="0.762" layer="25" font="vector" ratio="20" rot="R45" align="bottom-center"/>
+<attribute name="NAME" x="16.959015625" y="18.600984375" size="0.762" layer="25" font="vector" ratio="20" align="bottom-center"/>
 <attribute name="PROD_ID" value="IC-09069" x="16.51" y="19.05" size="1.778" layer="27" rot="R45" display="off"/>
 <attribute name="VALUE" x="21.000128125" y="14.559871875" size="0.6096" layer="27" font="vector" ratio="20" rot="R45" align="bottom-center"/>
@@
 </element>
 <element name="BUZ" library="testpad" library_urn="urn:adsk.eagle:library:385" package="B2,54" package3d_urn="urn:adsk.eagle:package:27948/1" value="TPB2,54" x="8.89" y="29.718" smashed="yes" rot="R90">
-<attribute name="NAME" x="6.731" y="31.242" size="0.762" layer="25" font="vector" ratio="10" rot="R270"/>
+<attribute name="NAME" x="7.112" y="31.369" size="0.762" layer="25" font="vector" ratio="10" rot="R180"/>
 <attribute name="TP_SIGNAL_NAME" value="" x="12.065" y="28.448" size="1" layer="37" rot="R90"/>
 <attribute name="VALUE" x="10.287" y="28.448" size="0.0254" layer="27" rot="R90"/>
@@
 <element name="C7" library="SparkFun-Capacitors" library_urn="urn:adsk.eagle:library:510" package="0603" package3d_urn="urn:adsk.eagle:package:37414/1" value="18pF" x="7.62" y="8.89" rot="MR0">
 <attribute name="PROD_ID" value="CAP-00867" x="7.62" y="8.89" size="1.778" layer="28" rot="MR0" display="off"/>
+</element>
+<element name="G" library="testpad" library_urn="urn:adsk.eagle:library:385" package="B1,27" package3d_urn="urn:adsk.eagle:package:27944/1" value="TPB1,27" x="13.97" y="27.94" smashed="yes">
+<attribute name="NAME" x="14.605" y="28.956" size="0.762" layer="25" ratio="10"/>
+<attribute name="TP_SIGNAL_NAME" value="" x="13.335" y="26.035" size="1" layer="37"/>
+<attribute name="VALUE" x="13.335" y="27.178" size="0.0254" layer="27"/>
+</element>
+<element name="5V" library="testpad" library_urn="urn:adsk.eagle:library:385" package="B1,27" package3d_urn="urn:adsk.eagle:package:27944/1" value="TPB1,27" x="13.97" y="30.48" smashed="yes">
+<attribute name="NAME" x="14.605" y="31.496" size="0.762" layer="25" font="vector" ratio="10"/>
+<attribute name="TP_SIGNAL_NAME" value="" x="13.335" y="28.575" size="1" layer="37"/>
+<attribute name="VALUE" x="13.335" y="29.718" size="0.0254" layer="27"/>
 </element>
 </elements>
@@
 <via x="11.43" y="8.89" extent="1-16" drill="0.35"/>
 <via x="15.24" y="20.32" extent="1-16" drill="0.35"/>
+<contactref element="G" pad="TP"/>
+<via x="-3.81" y="29.21" extent="1-16" drill="0.35"/>
+<via x="-3.81" y="27.94" extent="1-16" drill="0.35"/>
 </signal>
 <signal name="RED">
@@
 <wire x1="14.94" y1="30.42" x2="14.9" y2="30.48" width="0.3" layer="16"/>
 <via x="20.25" y="19.53" extent="1-16" drill="0.35"/>
+<contactref element="5V" pad="TP"/>
+<wire x1="16.51" y1="30.48" x2="13.97" y2="30.48" width="0.3" layer="1"/>
+<wire x1="14.9" y1="30.48" x2="16.51" y2="30.48" width="0.3" layer="16"/>
+<via x="16.51" y="30.48" extent="1-16" drill="0.35"/>
 </signal>
 <signal name="SCL">

Commit message: small fix
Parts:
- moved SW 3.59 mm to (20.3, 16.5)
Routing:
- net N$2: track 4.09 -> 5.36 mm
Changed lines of the file:
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@@
 <attribute name="VALUE" x="10.16" y="14.478" size="0.6096" layer="27" font="vector" ratio="20" rot="R180" align="top-center"/>
 </element>
-<element name="SW" library="testpad" library_urn="urn:adsk.eagle:library:385" package="B1,27" package3d_urn="urn:adsk.eagle:package:27944/1" value="TPB1,27" x="22.86" y="13.97" smashed="yes" rot="MR180">
-<attribute name="NAME" x="22.225" y="12.954" size="0.762" layer="26" font="vector" ratio="10" rot="MR180"/>
-<attribute name="TP_SIGNAL_NAME" value="" x="22.225" y="15.875" size="1" layer="38" rot="MR180"/>
-<attribute name="VALUE" x="22.225" y="14.732" size="0.0254" layer="28" rot="MR180"/>
+<element name="SW" library="testpad" library_urn="urn:adsk.eagle:library:385" package="B1,27" package3d_urn="urn:adsk.eagle:package:27944/1" value="TPB1,27" x="20.32" y="16.51" smashed="yes" rot="MR180">
+<attribute name="NAME" x="19.685" y="15.494" size="0.762" layer="26" font="vector" ratio="10" rot="MR180"/>
+<attribute name="TP_SIGNAL_NAME" value="" x="19.685" y="18.415" size="1" layer="38" rot="MR180"/>
+<attribute name="VALUE" x="19.685" y="17.272" size="0.0254" layer="28" rot="MR180"/>
 </element>
 <element name="LM1117" library="lm1117_10" package="SOT223" value="LM1117MP-5.0" x="8.89" y="15.24" smashed="yes" rot="MR0">
@@
 <wire x1="21.33" y1="14.76" x2="20.34" y2="15.75" width="0.2" layer="1"/>
 <wire x1="21.96" y1="14.76" x2="21.33" y2="14.76" width="0.2" layer="1"/>
-<wire x1="22.68" y1="14.04" x2="21.96" y2="14.76" width="0.2" layer="16"/>
-<wire x1="22.86" y1="14.04" x2="22.68" y2="14.04" width="0.2" layer="16"/>
+<wire x1="21.77" y1="15.17" x2="21.96" y2="14.76" width="0.2" layer="16"/>
+<wire x1="20.32" y1="16.58" x2="21.77" y2="15.17" width="0.2" layer="16"/>
 <wire x1="19.89" y1="16.29" x2="19.82816875" y2="16.297515625" width="0.2" layer="1"/>
-<wire x1="22.86" y1="14.04" x2="22.86" y2="13.97" width="0.2" layer="16"/>
+<wire x1="20.32" y1="16.58" x2="20.32" y2="16.51" width="0.2" layer="16"/>
 <via x="21.96" y="14.76" extent="1-16" drill="0.35"/>
 </signal>
