File: PCB Files/square Rev3.brd (EAGLE design)
At the start: 47 x 30.5 mm, 36 parts, among them Y1 16MHz

Commit message: PCB updates
Parts:
- C1: value 100nF -> 0.1uF
Changed lines of the file:
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@@
 <drawing>
 <settings>
-<setting alwaysvectorfont="yes"/>
+<setting alwaysvectorfont="no"/>
 <setting verticaltext="up"/>
 </settings>
@@
 </element>
 <element name="U3V12F9" library="SparkFun-Connectors" library_urn="urn:adsk.eagle:library:513" package="1X03" package3d_urn="urn:adsk.eagle:package:38063/1" value="" x="29.21" y="24.13" rot="MR0"/>
-<element name="C1" library="SparkFun-Capacitors" library_urn="urn:adsk.eagle:library:510" package="0603" package3d_urn="urn:adsk.eagle:package:37414/1" value="100nF" x="26.67" y="19.05" smashed="yes">
+<element name="C1" library="SparkFun-Capacitors" library_urn="urn:adsk.eagle:library:510" package="0603" package3d_urn="urn:adsk.eagle:package:37414/1" value="0.1uF" x="26.67" y="19.05" smashed="yes">
 <attribute name="NAME" x="26.67" y="19.812" size="0.762" layer="25" font="vector" ratio="10" align="bottom-center"/>
 <attribute name="PROD_ID" value="CAP-00867" x="26.67" y="19.05" size="1.778" layer="27" display="off"/>
